File: PCB/TeensyLC_DRV8871_MPRLS_Qwiic_v01/TeensyLC_DRV8871_MPRLS_Qwiic_v01.kicad_pcb (KiCad board)
At the start: 2 copper layers, 36.8 x 79.4 mm, 17 parts

Commit message: updated PCB
Parts:
- R1-330: renamed from R1-220; footprint Resistor_THT:R_Axial_DIN0207_L6.3mm_D2.5mm_P7.62mm_Horizontal -> Resistor_THT:R_Axial_DIN0207_L6.3mm_D2.5mm_P10.16mm_Horizontal
- R2-100: renamed from R2-220; footprint Resistor_THT:R_Axial_DIN0207_L6.3mm_D2.5mm_P7.62mm_Horizontal -> Resistor_THT:R_Axial_DIN0207_L6.3mm_D2.5mm_P10.16mm_Horizontal
- R3-4.7k, R4-4.7k: footprint Resistor_THT:R_Axial_DIN0207_L6.3mm_D2.5mm_P7.62mm_Horizontal -> Resistor_THT:R_Axial_DIN0207_L6.3mm_D2.5mm_P10.16mm_Horizontal
- moved R4-4.7k 7.24 mm to (44.5, 43.2), turned to 0 degrees
- moved R3-4.7k 3.70 mm to (44.5, 39.4), turned to 0 degrees
- moved R2-100 0.63 mm to (31.8, 43.2)
- renumbered D1 to D1-RED, D2 to D2_GRE
Routing:
- net /SCL0: track 18.8 -> 46.6 mm, vias 0 -> 2
- net /3V3: track 97.9 -> 122.4 mm
- net /SDA0: track 15.7 -> 26.8 mm
- net /SCL1: track 32.4 -> 26.9 mm
- net /SDA1: track 32.9 -> 29.9 mm
- net GND: track 2.12 -> 0.00 mm
- net /VIN: track 40.2 -> 42.0 mm
